File: Electronics/PCB/Supersonic Quantumbox/Supersonic Quantumbox.kicad_sch (KiCad schematic)
At the start: 5 parts

Commit message: Develop PCB
Parts:
- added C1: 100n, symbol Device:C
- added C10, C7, C8, C9: 10uF, symbol Device:C_Small
- added C2, C3: 10uF, symbol Device:C
- added C4, C5, C6, C? (x2): 100n, symbol Device:C_Small
- added C? (x4): (no value), symbol Device:C_Small
- added C?: 2.2uF, symbol Device:C_Small
- added R1, R2: 2M2, symbol Device:R
- added R3: 100K, symbol Device:R
- added R4: 220K, symbol Device:R
- added R5, R6, R7: 10K, symbol Device:R_Small
- added R?: 470, symbol Device:R_Small
- added R?: (no value), symbol Device:R_Small
- added RV1, RV2, RV3, RV4, RV5, RV6: R_Potentiometer, GustavsGlobalLibrary:PBD12 potentiometer, symbol Device:R_Potentiometer
- added U1: Input_jack, GustavsGlobalLibrary:Mono jack SYS212, symbol GlobalSymbolLibrary:Mono_jack
- added U2: TL071, Package_SO:SOIC-8_3.9x4.9mm_P1.27mm, symbol Amplifier_Operational:TL071
- added U7: PCM5100, Package_SO:TSSOP-20_4.4x6.5mm_P0.65mm, symbol Audio:PCM5100
- added U8: Output_jack, GustavsGlobalLibrary:Mono jack SYS212, symbol GlobalSymbolLibrary:Mono_jack
- J1: renamed from J?; value (none) -> USB_C_Receptacle_USB2.0; footprint (none) -> Connector_USB:USB_C_Receptacle_HRO_TYPE-C-31-M-12
- U3: renamed from U?; value (none) -> PCM1808PWR; footprint (none) -> GustavsGlobalLibrary:SOP65P640X120-14N
- U4: renamed from U?; value (none) -> AZ1117-5.0; footprint (none) -> Package_TO_SOT_SMD:TO-252-2
- U5: renamed from U?; value (none) -> ESP32-S2-WROVER-I; footprint (none) -> RF_Module:ESP32-S2-WROVER
- U6: renamed from U?; value (none) -> AZ1117-3.3; footprint (none) -> Package_TO_SOT_SMD:SOT-223-3_TabPin2
Connections:
- net +3V3: now also U3.4 (VDD), C10.2, C5.1, C?.1, C?.2, RV1.3, RV2.3, RV3.3, RV4.3, RV5.3, RV6.3, U7.1 (CPVDD), U7.10 (DEMP), U7.11 (FLT), U7.17 (XSMT), U7.20 (DVDD), U7.8 (AVDD)
- net +5V: now also U3.3 (VCC), C4.1, C8.2, C9.2
- net +9V: now also C7.2, R1.1, U2.7 (V+)
- net GNDREF: now also U3.2 (AGND), U3.5 (DGND), C10.1, C2.1, C4.2, C5.2, C6.1, C7.1, C8.1, C9.1, C?.1, C?.2, C?.2, C?.2, C?.2, C?.2, R2.2, R5.1, R6.1, R7.1, RV1.1, RV2.1, RV3.1, RV4.1, RV5.1, RV6.1, U1.2 (GND), U2.4 (V-), U7.12 (SCK), U7.16 (FMT), U7.19 (DGND), U7.3 (CPGND), U7.9 (AGND), U8.2 (GND)
- net at U3.1 (VREF): now also C6.2
- net at U3.10 (MD0): now also R6.2
- net at U3.11 (MD1): now also R7.2
- net at U3.12 (FMT): now also R5.2
- net at U3.13 (VINL): now also U3.14 (VINR), C3.2
- net IO0: now reaches U3.6 (SCKI)
- net IO0: now also U5.3 (IO00)
- net LRCK: now reaches U3.7 (LRCK)
- net LRCK: now also U5.10 (IO07), U7.15 (LRCK)
- net BCK: now reaches U3.8 (BCK)
- net BCK: now also U5.7 (IO04), U7.13 (BCK)
- net at U3.9 (DOUT): now also U5.21 (IO18)
- net DIN: now reaches U5.20 (IO17)
- net DIN: now also U7.14 (DIN)
- new net: C3.1, R4.2, U2.6
- new net: C2.2, R3.1
- new net: R3.2, R4.1, U2.2 (-)
- new net: C1.2, R1.2, R2.1, U2.3 (+)
- new net: C?.1, U7.2 (CAPP)
- new net: C?.2, U7.4 (CAPM)
- new net: R?.1, U7.7 (OUTR)
- new net: C?.1, R?.2, R?.2
- new net: C?.1, U7.5 (VNEG)
- new net: R?.1, U7.6 (OUTL)
- new net: C?.1, C?.1, U7.18 (LDOO)
- new net Input_signal: C1.1, U1.1 (Signal)
- new net Output_signal: U8.1 (Signal)
- new net Pot1: RV1.2
- new net Pot2: RV2.2
- new net Pot3: RV3.2
- new net Pot4: RV4.2
- new net Pot5: RV5.2
- new net Pot6: RV6.2
Other:
- moved on the sheet: J1, U3, U4, U5, U6

Commit message: Start work on PCB
Parts:
- added C11, C12, C20: 100n, Capacitor_SMD:C_0805_2012Metric_Pad1.18x1.45mm_HandSolder, symbol Device:C_Small
- added C21: 10uF, Capacitor_SMD:C_1206_3216Metric, symbol Device:C_Small
- added J2: Barrel_Jack_Switch, Connector_BarrelJack:BarrelJack_Horizontal, symbol Connector:Barrel_Jack_Switch
- added O1: 128x64_OLED, SupersonicQuantumbox:128x64OLED, symbol SupersonicQuantumbox:128x64_OLED
- added R11, R12: 5.1K, Resistor_SMD:R_0805_2012Metric_Pad1.20x1.40mm_HandSolder, symbol Device:R_Small
- added R8: 10K, Resistor_SMD:R_0805_2012Metric_Pad1.20x1.40mm_HandSolder, symbol Device:R_Small
- added SW1: RESET, Button_Switch_SMD:SW_Push_1P1T_NO_6x6mm_H9.5mm, symbol Switch:SW_Push
- added SW2: BOOT, Button_Switch_SMD:SW_Push_1P1T_NO_6x6mm_H9.5mm, symbol Switch:SW_Push
- C1, C4, C5, C6: footprint (none) -> Capacitor_SMD:C_0805_2012Metric_Pad1.18x1.45mm_HandSolder
- C10, C2, C3, C7, C8, C9: footprint (none) -> Capacitor_SMD:C_1206_3216Metric
- C13, C14: renamed from C?; footprint (none) -> Capacitor_SMD:C_0805_2012Metric_Pad1.18x1.45mm_HandSolder
- C15: renamed from C?; value (none) -> 2.2uF; footprint (none) -> Capacitor_SMD:C_1206_3216Metric
- C16: renamed from C?; footprint (none) -> Capacitor_SMD:C_1206_3216Metric
- C17: renamed from C?; value (none) -> 100n; footprint (none) -> Capacitor_SMD:C_0805_2012Metric_Pad1.18x1.45mm_HandSolder
- C18: renamed from C?; value (none) -> 10uF; footprint (none) -> Capacitor_SMD:C_1206_3216Metric
- C19: renamed from C?; value (none) -> 2.2n; footprint (none) -> Capacitor_SMD:C_0805_2012Metric_Pad1.18x1.45mm_HandSolder
- R1, R2, R3, R4, R5, R6, R7: footprint (none) -> Resistor_SMD:R_0805_2012Metric_Pad1.20x1.40mm_HandSolder
- R10: renamed from R?; footprint (none) -> Resistor_SMD:R_0805_2012Metric_Pad1.20x1.40mm_HandSolder
- R9: renamed from R?; value (none) -> 470; footprint (none) -> Resistor_SMD:R_0805_2012Metric_Pad1.20x1.40mm_HandSolder
Connections:
- net +3V3: now also C11.2, O1.2 (VCC), R8.2
- net +9V: now also C20.1, J2.1
- net BCK: now also U5.16 (IO13); no longer U5.7 (IO04)
- net DIN: now also U5.21 (IO18); no longer U5.20 (IO17)
- net GNDREF: now also C11.1, C12.1, C20.2, C21.1, J2.2, O1.1 (GND), R11.2, R12.2, SW1.1, SW2.1
- net IO0: now also SW2.2
- net LRCK: now also U5.17 (IO14); no longer U5.10 (IO07)
- net Pot1: now also U5.4 (IO01)
- net Pot2: now also U5.5 (IO02)
- net Pot3: now also U5.6 (IO03)
- net Pot4: now also U5.7 (IO04)
- net Pot5: now also U5.8 (IO05)
- net Pot6: now also U5.9 (IO06)
- net USB_D+: now also U5.23 (USB_D+)
- net USB_D-: now also U5.22 (USB_D-)
- net at C6.2, U3.1 (VREF): now also C21.2
- net at U3.9 (DOUT): now also U5.20 (IO17); no longer U5.21 (IO18)
- net SDA: now reaches U5.14 (IO11)
- net SDA: now also O1.4 (SDA)
- net SCL: now reaches U5.15 (IO12)
- net SCL: now also O1.3 (SCL)
- net EN: now reaches U5.41 (EN)
- net EN: now also C12.2, R8.1, SW1.2
- net at J1.A5 (CC1): now also R11.1
- net at J1.B5 (CC2): now also R12.1
- no-connect marks 0 -> 3
Other:
- note added: "3V3 LDO"
- note added: "5V LDO"
- note added: "ADC"
- note added: "ADC2 on GPIO 11-18 Not usable during wifi"
- note added: "Boot select"
- note added: "DAC"
- note added: "DC input"
- note added: "ESP Reset"
- note added: "ESP32-s2"
- note added: "GPIOs"
- note added: "Input buffering"
- note added: "Potentiometers"
- note added: "Screen"
- note added: "USB-C Jack"
- moved on the sheet: C1, C10, C13, C14, C15, C16, C17, C18, C19, C2, C3, C4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

Commit message: Change PCB layout
Parts:
- added D1, D2: WS2812B, LED_SMD:LED_WS2812B_PLCC4_5.0x5.0mm_P3.2mm, symbol LED:WS2812B
- added R13, R14: 10K, Resistor_SMD:R_0805_2012Metric_Pad1.20x1.40mm_HandSolder, symbol Device:R_Small
- added SW3: RotaryEncoder_Switch, Rotary_Encoder:RotaryEncoder_Alps_EC12E-Switch_Vertical_H20mm, symbol Device:RotaryEncoder_Switch
Connections:
- net +3V3: now also R13.2, R14.2
- net +5V: now also D1.1 (VDD), D2.1 (VDD)
- net GNDREF: now also D1.3 (VSS), D2.3 (VSS), SW3.C, SW3.S1
- net ENC_SW: now reaches U5.10 (IO07)
- net ENC_SW: now also SW3.S2
- net ENC_B: now reaches U5.11 (IO08)
- net ENC_B: now also R14.1, SW3.B
- net ENC_A: now reaches U5.12 (IO09)
- net ENC_A: now also R13.1, SW3.A
- net NEOP: now reaches U5.13 (IO10)
- net NEOP: now also D1.4 (DIN)
- new net: D1.2 (DOUT), D2.4 (DIN)
Other:
- note added: "Rotary Encoder"

Commit message: Routing
Parts:
- added C22, C23: 100n, Capacitor_SMD:C_0805_2012Metric_Pad1.18x1.45mm_HandSolder, symbol Device:C_Small
- added D3: LED2, symbol Device:LED
- added D4: LED1, symbol Device:LED
- added D5: PWR_LED, LED_SMD:LED_0805_2012Metric_Pad1.15x1.40mm_HandSolder, symbol Device:LED
- added H1, H2, H3, H4: M3, MountingHole:MountingHole_3.2mm_M3_Pad_Via, symbol Mechanical:MountingHole_Pad
- added J3: UART, Connector_PinHeader_2.54mm:PinHeader_1x02_P2.54mm_Vertical, symbol Connector:Conn_01x02_Male
- added J4: GPIO2, Connector_PinSocket_2.54mm:PinSocket_1x05_P2.54mm_Vertical, symbol Connector:Conn_01x05_Male
- added J5: GPIO1, Connector_PinSocket_2.54mm:PinSocket_1x05_P2.54mm_Vertical, symbol Connector:Conn_01x05_Male
- added JP1: GND_JMP, Jumper:SolderJumper-2_P1.3mm_Open_TrianglePad1.0x1.5mm, symbol Jumper:SolderJumper_2_Open
- added R15: R_LED, Resistor_SMD:R_0805_2012Metric_Pad1.20x1.40mm_HandSolder, symbol Device:R_Small
- added SW4: SW_DPDT_x2, symbol Switch:SW_DPDT_x2
- R5, R7: value 10K -> R_LED
- U1, U8: footprint GustavsGlobalLibrary:Mono jack SYS212 -> SupersonicQuantumbox:MonoJack-SYS212
Connections:
- net +3V3: now also D1.1 (VDD), D2.1 (VDD), C22.2, C23.2, J4.1 (Pin_1)
- net +5V: now also D5.2 (A); no longer D1.1 (VDD), D2.1 (VDD)
- net BCK: now also U5.18 (IO15); no longer U5.16 (IO13)
- net DIN: now also U5.20 (IO17); no longer U5.21 (IO18)
- net ENC_A: now also U5.14 (IO11); no longer U5.12 (IO09)
- net ENC_B: now also U5.13 (IO10); no longer U5.11 (IO08)
- net ENC_SW: now also U5.15 (IO12); no longer U5.10 (IO07)
- net GNDREF: now also C22.1, C23.1, D3.1 (K), D4.1 (K), J5.5 (Pin_5), JP1.1 (A), R15.1; no longer R5.1, R7.1
- net LRCK: now also U5.21 (IO18); no longer U5.17 (IO14)
- net NEOP: now also U5.8 (IO05); no longer U5.13 (IO10)
- net Pot5: now also U5.12 (IO09); no longer U5.8 (IO05)
- net Pot6: now also U5.11 (IO08); no longer U5.9 (IO06)
- net SCL: now also U5.9 (IO06); no longer U5.15 (IO12)
- net SDA: now also U5.10 (IO07); no longer U5.14 (IO11)
- net at R7.2: now also D4.2 (A); no longer U3.11 (MD1)
- net at R6.2, U3.10 (MD0): now also U3.11 (MD1), U3.12 (FMT)
- net DSP_OUT: now reaches C19.1, R10.2, R9.2
- net DSP_OUT: now also SW4.4 (A)
- net at R5.2: now also D3.2 (A); no longer U3.12 (FMT)
- net DOUT: now reaches U3.9 (DOUT)
- net DOUT: now also U5.19 (IO16); no longer U5.20 (IO17)
- net IO33: now reaches U5.27 (IO33)
- net IO33: now also J5.4 (Pin_4)
- net IO34: now reaches U5.28 (IO34)
- net IO34: now also J5.3 (Pin_3)
- net IO35: now reaches U5.29 (IO35)
- net IO35: now also J5.2 (Pin_2)
- net IO36: now reaches U5.30 (IO36)
- net IO36: now also J5.1 (Pin_1)
- net IO37: now reaches U5.31 (IO37)
- net IO37: now also J4.5 (Pin_5)
- net IO38: now reaches U5.32 (IO38)
- net IO38: now also J4.4 (Pin_4)
- net IO39: now reaches U5.33 (IO39)
- net IO39: now also J4.3 (Pin_3)
- net IO40: now reaches U5.34 (IO40)
- net IO40: now also J4.2 (Pin_2)
- net TX: now reaches U5.37 (TXD0)
- net TX: now also J3.2 (Pin_2)
- net RX: now reaches U5.38 (RXD0)
- net RX: now also J3.1 (Pin_1)
- net Input_signal renamed DSP_IN
- net DSP_IN: now also SW4.1 (A); no longer U1.1 (Signal)
- net Output_signal renamed JACK_OUT
- net JACK_OUT: now also SW4.5 (B)
- new net: H1.1, JP1.2 (B)
- new net: D5.1 (K), R15.2
- new net BYPASS: SW4.3 (C), SW4.6 (C)
- new net JACK_IN: SW4.2 (B), U1.1 (Signal)
- new net LED1: R7.1, U5.16 (IO13)
- new net LED2: R5.1, U5.17 (IO14)
- no-connect marks 3 -> 9
Other:
- note added: "LED filaments"
- note added: "Mounting holes"
- note added: "Neopixels"
- note added: "Power LED"
- note added: "True bypass"
- note removed: "GPIOs"
- moved on the sheet: C1, C13, C14, C15, C16, C17, C18, C19, C2, C20, C3, R1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

Commit message: Begin PWR tracing
Changed lines of the file:
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@@
       (effects (font (size 1.27 1.27)) hide)
     )
-    (property "Value" "+3V3" (id 1) (at 273.05 134.6199 90)
+    (property "Value" "+3V3" (id 1) (at 270.51 134.6199 90)
       (effects (font (size 1.27 1.27)) (justify right))
     )
@@
       (effects (font (size 1.27 1.27)) hide)
     )
+    (pin "1")
+    (pin "2")
+    (pin "3")
     (pin "4")
     (pin "5")
@@
     (pin "2")
     (pin "3")
+    (pin "4")
+    (pin "5")
+    (pin "6")
   )
   (symbol (lib_id "Switch:SW_Push") (at 237.49 69.85 0) (unit 1)
@@
     )
     (path "/2617224a-f69a-48d1-b2a5-2492a163990a"
-      (reference "D3") (unit 1) (value "LED2") (footprint "")
+      (reference "D3") (unit 1) (value "LED2") (footprint "SupersonicQuantumbox:38 mm LED")
     )
     (path "/5ef8d7b2-8fc8-4f84-ae46-e8f6a43a45c0"
-      (reference "D4") (unit 1) (value "LED1") (footprint "")
+      (reference "D4") (unit 1) (value "LED1") (footprint "SupersonicQuantumbox:38 mm LED")
     )
     (path "/3359374b-bccb-4c0d-8386-f383440986f1"
@@
     )
     (path "/2c8bc3cc-6dd3-4f97-bd0d-8eec23ff3b4e"
-      (reference "SW4") (unit 2) (value "SW_DPDT_x2") (footprint "")
+      (reference "SW4") (unit 2) (value "SW_DPDT_x2") (footprint "SupersonicQuantumbox:Stomp_switch")
     )
     (path "/c3e1c4c6-64d8-4eb6-86eb-759cbb00d7a2"

Commit message: Final touches
Parts:
- C19: value 2.2n -> 22n
- D3, D4: footprint (none) -> SupersonicQuantumbox:38 mm LED
- R10, R9: value 470 -> 470R
- SW4: footprint (none) -> SupersonicQuantumbox:Stomp_switch
