File: Electronics/PCB/Supersonic Quantumbox/Supersonic Quantumbox.kicad_sch (KiCad schematic)
At the start: 63 parts, among them IC1 AK4558EN, J1 USB_C_Receptacle_USB2.0, J2 Conn_01x12_Pin, J6 Barrel_Jack_Switch, SW1 RESET, SW2 BOOT, SW3 RotaryEncoder_Switch, SW4 SW_DPDT_x2, U1 Input_jack, U2 AZ1117-5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

Commit message: Routing
Connections:
- net +3V3: now also D5.2 (A)
- net +5V: no longer D5.2 (A)
- no-connect marks 9 -> 12
Changed lines of the file:
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@@
   (junction (at 50.8 110.49) (diameter 0) (color 0 0 0 0)
   )
+  (no_connect (at 165.1 31.75))
+  (no_connect (at 283.21 152.4))
   (no_connect (at 196.85 25.4))
   (no_connect (at 217.17 25.4))
@@
   (no_connect (at 210.82 50.8))
   (no_connect (at 292.1 127))
+  (no_connect (at 280.67 30.48))
   (wire (pts (xy 284.48 142.24) (xy 292.1 142.24))
     (stroke (width 0) (type default))
@@
     )
   )
-  (symbol (lib_id "power:+5V") (at 142.24 187.96 0) (unit 1)
-    (in_bom yes) (on_board yes) (dnp no) (fields_autoplaced)
-    (property "Reference" "#PWR024" (at 142.24 191.77 0)
-      (effects (font (size 1.27 1.27)) hide)
-    )
-    (property "Value" "+5V" (at 143.637 187.169 0)
-      (effects (font (size 1.27 1.27)) (justify left))
-    )
-    (property "Footprint" "" (at 142.24 187.96 0)
-      (effects (font (size 1.27 1.27)) hide)
-    )
-    (property "Datasheet" "" (at 142.24 187.96 0)
-      (effects (font (size 1.27 1.27)) hide)
-    )
-    (pin "1")
-    (instances
-      (project "Supersonic Quantumbox"
-        (path "/0ee88c70-b4a6-4a69-8494-c8cddbda5aef"
-          (reference "#PWR024") (unit 1)
-        )
-      )
-    )
-  )
   (symbol (lib_id "power:GNDREF") (at 328.93 96.52 0) (unit 1)
     (in_bom yes) (on_board yes) (dnp no)
@@
     )
   )
-  (symbol (lib_name "+3V3_1") (lib_id "power:+3V3") (at 201.93 119.38 0) (unit 1)
+  (symbol (lib_id "power:+3V3") (at 201.93 119.38 0) (unit 1)
     (in_bom yes) (on_board yes) (dnp no)
     (property "Reference" "#PWR012" (at 201.93 123.19 0)
@@
     )
   )
-  (symbol (lib_name "+3V3_1") (lib_id "power:+3V3") (at 153.67 162.56 0) (unit 1)
+  (symbol (lib_id "power:+3V3") (at 153.67 162.56 0) (unit 1)
     (in_bom yes) (on_board yes) (dnp no)
     (property "Reference" "#PWR030" (at 153.67 166.37 0)
@@
     )
   )
+  (symbol (lib_id "power:+3V3") (at 142.24 187.96 0) (unit 1)
+    (in_bom yes) (on_board yes) (dnp no)
+    (property "Reference" "#PWR020" (at 142.24 191.77 0)
+      (effects (font (size 1.27 1.27)) hide)
+    )
+    (property "Value" "+3V3" (at 140.97 184.15 0)
+      (effects (font (size 1.27 1.27)))
+    )
+    (property "Footprint" "" (at 142.24 187.96 0)
+      (effects (font (size 1.27 1.27)) hide)
+    )
+    (property "Datasheet" "" (at 142.24 187.96 0)
+      (effects (font (size 1.27 1.27)) hide)
+    )
+    (pin "1")
+    (instances
+      (project "Supersonic Quantumbox"
+        (path "/0ee88c70-b4a6-4a69-8494-c8cddbda5aef"
+          (reference "#PWR020") (unit 1)
+        )
+      )
+    )
+  )
   (symbol (lib_id "Device:C_Small") (at 118.11 127 180) (unit 1)
     (in_bom yes) (on_board yes) (dnp no)
@@
     )
   )
-  (symbol (lib_name "+3V3_1") (lib_id "power:+3V3") (at 167.64 106.68 0) (unit 1)
+  (symbol (lib_id "power:+3V3") (at 167.64 106.68 0) (unit 1)
     (in_bom yes) (on_board yes) (dnp no)
     (property "Reference" "#PWR031" (at 167.64 110.49 0)
@@
     )
   )
-  (symbol (lib_name "+3V3_1") (lib_id "power:+3V3") (at 152.4 109.22 0) (unit 1)
+  (symbol (lib_id "power:+3V3") (at 152.4 109.22 0) (unit 1)
     (in_bom yes) (on_board yes) (dnp no)
     (property "Reference" "#PWR011" (at 152.4 113.03 0)

Commit message: Routing complete
Parts:
- removed C22, C23: 100n, Capacitor_SMD:C_0603_1608Metric, symbol Device:C_Small
- removed D1, D2: WS2812B, LED_SMD:LED_WS2812B_PLCC4_5.0x5.0mm_P3.2mm, symbol LED:WS2812B
Connections:
- no-connect marks 12 -> 11
Other:
- note removed: "Neopixels"

Commit message: PCB finished
Parts:
- added J3: Conn_02x03_Counter_Clockwise, Connector_PinSocket_2.54mm:PinSocket_2x03_P2.54mm_Horizontal, symbol Connector_Generic:Conn_02x03_Odd_Even
Connections:
- net +3V3: now also J3.5 (Pin_5)
- net GNDREF: now also J3.2 (Pin_2)
- net IO41: now reaches U9.34 (IO41)
- net IO41: now also J3.3 (Pin_3)
- net IO42: now reaches U9.35 (IO42)
- net IO42: now also J3.1 (Pin_1)
- net IO2: now reaches U9.38 (IO2)
- net IO2: now also J3.6 (Pin_6)
- net IO1: now reaches U9.39 (IO1)
- net IO1: now also J3.4 (Pin_4)
- net NEOP: no longer names the net of U9.17 (IO9)
Other:
- note added: "Extension"
- moved on the sheet: C11, U9
