File: Electronics/PCB/Supersonic Quantumbox/Supersonic Quantumbox.kicad_pcb (KiCad board)
At the start: 2 copper layers, 80 x 150 mm, 76 parts, among them J1 USB_C_Receptacle_USB2.0, J2 Barrel_Jack_Switch, J3 UART, J4 GPIO2, J5 GPIO1, SW1 RESET, SW2 BOOT, SW3 RotaryEncoder_Switch, SW4 SW_DPDT_x2, U1 Input_jack, U2 TL071, U3 PCM1808PWR, U4 AZ1117-5.0, U5 ESP32-S2-WROVER-I, U6 AZ1117-3.3, U7 PCM5100, U8 Output_jack

Commit message: V2 schematic complete
Parts:
- removed C20: 100n, Capacitor_SMD:C_0805_2012Metric_Pad1.18x1.45mm_HandSolder
- removed C21: 10uF, Capacitor_SMD:C_1206_3216Metric
- removed D3: LED2, SupersonicQuantumbox:38 mm LED
- removed D4: LED1, SupersonicQuantumbox:38 mm LED
- removed G*** (x3): LOGO, LOGO
- removed J3: UART, Connector_PinHeader_2.54mm:PinHeader_1x02_P2.54mm_Vertical
- removed J4: GPIO2, Connector_PinSocket_2.54mm:PinSocket_1x05_P2.54mm_Vertical
- removed J5: GPIO1, Connector_PinSocket_2.54mm:PinSocket_1x05_P2.54mm_Vertical
- removed O1: 128x64_OLED, SupersonicQuantumbox:128x64OLED
- removed R2: 2M2, Resistor_SMD:R_0805_2012Metric_Pad1.20x1.40mm_HandSolder
- removed REF**: KiCad-Logo2_5mm_SilkScreen, Symbol:KiCad-Logo2_5mm_SilkScreen
- removed RV4, RV5, RV6: R_Potentiometer, GustavsGlobalLibrary:PBD12 potentiometer
- removed U3: PCM1808PWR, GustavsGlobalLibrary:SOP65P640X120-14N
- removed U7: PCM5100, Package_SO:TSSOP-20_4.4x6.5mm_P0.65mm
- added IC1: AK4558EN, SupersonicQuantumbox:QFN50P500X500X75-29N, B.Cu at (93.0, 103.0)
- added J6: Barrel_Jack_Switch, Connector_BarrelJack:BarrelJack_Horizontal, B.Cu at (115.0, 67.0)
- added R16: 10k, Resistor_SMD:R_0603_1608Metric, B.Cu at (101.0, 126.0)
- added R17: 1M, Resistor_SMD:R_0603_1608Metric, B.Cu at (109.0, 126.0)
- added U9: ESP32-S3-WROOM-1-N8R8, SupersonicQuantumbox:XCVR_ESP32S3WROOM1N8R8, B.Cu at (83.0, 86.0)
- C1: value 100n -> 0.1uF; footprint Capacitor_SMD:C_0805_2012Metric_Pad1.18x1.45mm_HandSolder -> Capacitor_THT:C_Rect_L10.3mm_W5.7mm_P7.50mm_MKS4
- C11, C12, C13, C17, C5: footprint Capacitor_SMD:C_0805_2012Metric_Pad1.18x1.45mm_HandSolder -> Capacitor_SMD:C_0603_1608Metric
- C14: value 100n -> 3.3uF; footprint Capacitor_SMD:C_0805_2012Metric_Pad1.18x1.45mm_HandSolder -> Capacitor_THT:C_Rect_L26.5mm_W10.5mm_P22.50mm_MKS4
- C15, C16: value 2.2uF -> 10uF
- C18: value 10uF -> BFC; footprint Capacitor_SMD:C_1206_3216Metric -> Capacitor_THT:CP_Radial_D6.3mm_P2.50mm
- C19: value 22n -> BFC; footprint Capacitor_SMD:C_0805_2012Metric_Pad1.18x1.45mm_HandSolder -> Capacitor_THT:CP_Radial_D6.3mm_P2.50mm
- C2, C3: value 10uF -> 3.3uF; footprint Capacitor_SMD:C_1206_3216Metric -> Capacitor_THT:C_Rect_L26.5mm_W10.5mm_P22.50mm_MKS4
- C22, C23: footprint Capacitor_SMD:C_0805_2012Metric_Pad1.18x1.45mm_HandSolder -> Capacitor_SMD:C_0603_1608Metric; moved to F.Cu
- C4, C6: value 100n -> 1u; footprint Capacitor_SMD:C_0805_2012Metric_Pad1.18x1.45mm_HandSolder -> Capacitor_SMD:C_0603_1608Metric
- H1, H2, H3, H4: value M3 -> M2; footprint MountingHole:MountingHole_3.2mm_M3_Pad_Via -> MountingHole:MountingHole_2.2mm_M2_Pad_Via
- J2: value Barrel_Jack_Switch -> Conn_01x12_Pin; footprint Connector_BarrelJack:BarrelJack_Horizontal -> Connector_FFC-FPC:TE_1-1734839-2_1x12-1MP_P0.5mm_Horizontal
- R1: value 2M2 -> 10k; footprint Resistor_SMD:R_0805_2012Metric_Pad1.20x1.40mm_HandSolder -> Resistor_SMD:R_0603_1608Metric
- R10: value 470R -> BL; footprint Resistor_SMD:R_0805_2012Metric_Pad1.20x1.40mm_HandSolder -> Resistor_SMD:R_0603_1608Metric
- R11, R12, R13, R14, R15, R3, R4, R8: footprint Resistor_SMD:R_0805_2012Metric_Pad1.20x1.40mm_HandSolder -> Resistor_SMD:R_0603_1608Metric
- R5, R7: value R_LED -> 10K; footprint Resistor_SMD:R_0805_2012Metric_Pad1.20x1.40mm_HandSolder -> Resistor_SMD:R_0603_1608Metric
- R6: value 10K -> 10k; footprint Resistor_SMD:R_0805_2012Metric_Pad1.20x1.40mm_HandSolder -> Resistor_SMD:R_0603_1608Metric
- R9: value 470R -> 10K; footprint Resistor_SMD:R_0805_2012Metric_Pad1.20x1.40mm_HandSolder -> Resistor_SMD:R_0603_1608Metric
- RV1, RV2, RV3: footprint GustavsGlobalLibrary:PBD12 potentiometer -> Potentiometer_THT:Potentiometer_Alps_RK09K_Single_Vertical
- SW1, SW2: footprint Button_Switch_SMD:SW_Push_1P1T_NO_6x6mm_H9.5mm -> Button_Switch_SMD:SW_SPST_EVQP7C
- SW4: footprint SupersonicQuantumbox:Stomp_switch -> SupersonicQuantumbox:SW_Push_2P2T_Toggle_MHPS2285
- U2: value TL071 -> AZ1117-5; footprint Package_SO:SOIC-8_3.9x4.9mm_P1.27mm -> Package_TO_SOT_SMD:SOT-223-3_TabPin2
- U4: value AZ1117-5.0 -> TPS7A2033; footprint Package_TO_SOT_SMD:TO-252-2 -> Package_TO_SOT_SMD:SOT-23-5
- U5: value ESP32-S2-WROVER-I -> LM6742; footprint RF_Module:ESP32-S2-WROVER -> Package_SO:SOIC-8_3.9x4.9mm_P1.27mm
- moved H4 128.1 mm to (137.0, 152.0)
- moved H3 126.6 mm to (73.0, 152.0)
- moved H2 114.5 mm to (137.0, 58.0)
- moved H1 112.8 mm to (73.0, 58.0)
- moved R9 102.7 mm to (81.0, 65.0), turned to 180 degrees
- moved C7 101.9 mm to (105.0, 130.0), turned to 180 degrees
- moved JP1 100.6 mm to (73.0, 64.3), turned to 90 degrees
- moved D2 93.5 mm to (52.5, 82.5)
- moved C23 93.2 mm to (55.0, 89.0), turned to 0 degrees
- moved C3 89.4 mm to (73.0, 114.0), turned to 0 degrees
- moved U2 89.4 mm to (120.0, 77.0), turned to -90 degrees
- moved R10 80.5 mm to (101.0, 84.0), turned to 180 degrees
- moved C11 80.3 mm to (74.0, 74.0), turned to 0 degrees
- moved C19 78.8 mm to (117.1, 86.0), turned to 0 degrees
- moved U4 69.8 mm to (118.0, 105.0), turned to -90 degrees
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Connections:
- C1 pad 2: Net-(C1-Pad2) -> Net-(U5A-+)
- C13 pad 2: +3V3 -> +3.3VA
- C14 pad 1: +3V3 -> /DSP_OUT
- C14 pad 2: GNDREF -> Net-(U5B--)
- C15 pad 1: Net-(C15-Pad1) -> GNDREF
- C15 pad 2: Net-(C15-Pad2) -> +5V
- C16 pad 1: Net-(C16-Pad1) -> GNDREF
- C16 pad 2: GNDREF -> +3.3VA
- C17 pad 1: Net-(C17-Pad1) -> +3.3VA
- C18 pad 1: Net-(C17-Pad1) -> +5V
- C19 pad 1: /DSP_OUT -> +5V
- C3 pad 2: Net-(C3-Pad2) -> /LINE_IN
- C4 pad 1: +5V -> Net-(IC1-VDD18)
- C5 pad 1: +3V3 -> GNDREF
- C5 pad 2: GNDREF -> +3V3
- C7 pad 2: +9V -> Net-(C7-Pad2)
- C8 pad 2: +5V -> +9V
- J2 pad 1: +9V -> GNDREF
- J2 pad 2: GNDREF -> Net-(J2-Pin_2)
- J2 pad 3: unconnected-(J2-Pad3) -> +3V3
- R1 pad 1: +9V -> +3.3VA
- R1 pad 2: Net-(C1-Pad2) -> Net-(C7-Pad2)
- R10 pad 1: Net-(R10-Pad1) -> GNDREF
- R10 pad 2: /DSP_OUT -> Net-(J2-Pin_2)
- R3 pad 2: Net-(R3-Pad2) -> Net-(U5A--)
- R4 pad 1: Net-(R3-Pad2) -> Net-(U5A--)
- R5 pad 1: /LED2 -> +3V3
- R5 pad 2: Net-(D3-Pad2) -> Net-(R5-Pad2)
- R6 pad 2: Net-(R6-Pad2) -> /DSP_OUT
- R7 pad 1: /LED1 -> +3V3
- R7 pad 2: Net-(D4-Pad2) -> Net-(R7-Pad2)
- R9 pad 1: Net-(R9-Pad1) -> +3V3
- R9 pad 2: /DSP_OUT -> Net-(R9-Pad2)
- RV1 pad 3: +3V3 -> Net-(R9-Pad2)
- RV2 pad 3: +3V3 -> Net-(R7-Pad2)
- RV3 pad 3: +3V3 -> Net-(R5-Pad2)
- U2 pad 1: unconnected-(U2-Pad1) -> GNDREF
- U2 pad 2: Net-(R3-Pad2) -> +5V
- U2 pad 3: Net-(C1-Pad2) -> +9V
- U4 pad 1: GNDREF -> +5V
- U4 pad 2: +5V -> GNDREF
- U4 pad 3: +9V -> +5V
- U5 pad 1: GNDREF -> Net-(C3-Pad1)
- U5 pad 2: +3V3 -> Net-(U5A--)
- U5 pad 3: /IO0 -> Net-(U5A-+)
- U5 pad 4: /Pot1 -> GNDREF
- U5 pad 5: /Pot2 -> Net-(IC1-LOUT)
- U5 pad 6: /Pot3 -> Net-(U5B--)
- U5 pad 7: /Pot4 -> Net-(U5B--)
- U5 pad 8: /NEOP -> +3.3VA
Routing:
- net +3V3: track 379.6 -> 0.00 mm, vias 9 -> 0
- net +9V: track 256.2 -> 0.00 mm
- net +5V: track 184.6 -> 0.00 mm, vias 2 -> 0
- net /EN: track 113.7 -> 0.00 mm, vias 4 -> 0
- net Net-(D3-Pad2): track 99.6 -> 0.00 mm, vias 4 -> 0
- net GNDREF: track 93.9 -> 0.00 mm, vias 227 -> 0
- net /BCK: track 91.4 -> 0.00 mm, vias 2 -> 0
- net /IO0: track 87.1 -> 0.00 mm, vias 2 -> 0
- net /Pot3: track 85.2 -> 0.00 mm
- net /LRCK: track 81.1 -> 0.00 mm, vias 2 -> 0
- net /SCL: track 78.5 -> 0.00 mm
- net /SDA: track 76.1 -> 0.00 mm
- net /Pot2: track 74.2 -> 0.00 mm
- net /Pot1: track 54.5 -> 0.00 mm
- net /Pot6: track 53.9 -> 0.00 mm
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- added copper zone on In1.Cu, net GNDREF
- added copper zone on In2.Cu, net GNDREF
- removed copper zone on B.Cu, net GNDREF
- removed copper zone on F.Cu, net GNDREF
Other:
- board size 80 x 150 mm -> 70 x 100 mm
- copper layers 2 -> 4
- board text removed: "+9V"
- board text removed: "2022 v1.0"
- board text removed: "3.3V"
- board text removed: "3V3"
- board text removed: "A. Anderson"
- board text removed: "BND"
- board text removed: "G. Abrahamsson"
- board text removed: "GND"
- board text removed: "IN"
- board text removed: "IO33"
- board text removed: "IO34"
- board text removed: "IO35"
- board text removed: "IO36"
- board text removed: "IO37"
- board text removed: "IO38"
- board text removed: "IO39"
- board text removed: "IO40"
- board text removed: "JLCJLCJLCJLC"
- board text removed: "OUT"
- board text removed: "Pot1"
- board text removed: "Pot2"
- board text removed: "Pot3"
- board text removed: "Pot4"
- board text removed: "Pot5"
- board text removed: "Pot6"
- board text removed: "RX"
- board text removed: "SCL"
- board text removed: "SDA"
- board text removed: "Supersonic Quantumbox"
- board text removed: "TX"

Commit message: Routing
Parts:
- moved R14 44.9 mm to (92.2, 74.2), turned to 0 degrees
- moved R13 44.4 mm to (88.8, 74.2), turned to 180 degrees
- moved C13 11.4 mm to (94.8, 107.0), turned to 180 degrees
- moved C1 7.49 mm to (114.3, 128.0), turned to 0 degrees
- moved C17 6.32 mm to (103.0, 114.0), turned to 180 degrees
- moved C11 4.26 mm to (78.2, 74.2)
- moved C12 3.76 mm to (81.8, 74.2)
- moved R8 3.26 mm to (85.2, 74.2)
- moved R9 2.06 mm to (81.5, 67.0), turned to 0 degrees
- moved R5 2.02 mm to (128.8, 67.0), turned to 0 degrees
- moved R7 2.02 mm to (105.2, 67.0), turned to 0 degrees
- moved R10 1.41 mm to (102.0, 85.0), turned to -90 degrees
- moved R11 1.03 mm to (129.0, 75.2)
- moved R12 0.96 mm to (128.9, 78.8)
- moved C6 0.75 mm to (91.2, 107.0)
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Connections:
- D5 pad 2: +5V -> +3V3
Routing:
- net +3V3: track 0.00 -> 123.9 mm, vias 0 -> 2
- net /IO0: track 0.00 -> 62.9 mm, vias 0 -> 2
- net /ENC_B: track 0.00 -> 62.2 mm, vias 0 -> 2
- net /ENC_A: track 0.00 -> 62.1 mm, vias 0 -> 2
- net +3.3VA: track 0.00 -> 57.8 mm, vias 0 -> 2
- net /Pot3: track 0.00 -> 50.5 mm, vias 0 -> 1
- net /ENC_SW: track 0.00 -> 50.4 mm, vias 0 -> 1
- net Net-(C3-Pad1): track 0.00 -> 43.1 mm, vias 0 -> 1
- net /DSP_OUT: track 0.00 -> 41.6 mm
- net /USB_D-: track 5.00 -> 43.9 mm, vias 0 -> 2
- net /USB_D+: track 4.80 -> 42.6 mm, vias 0 -> 2
- net /Pot2: track 0.00 -> 34.1 mm, vias 0 -> 1
- net /JACK_IN: track 0.00 -> 31.1 mm
- net /JACK_OUT: track 0.00 -> 27.6 mm
- net Net-(U5A-+): track 0.00 -> 22.9 mm
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- added copper zone on B.Cu, net +5V
- added copper zone on B.Cu, net GNDREF

Commit message: Routing complete
Parts:
- removed C22, C23: 100n, Capacitor_SMD:C_0603_1608Metric
- removed D1, D2: WS2812B, LED_SMD:LED_WS2812B_PLCC4_5.0x5.0mm_P3.2mm
- moved D5 3.25 mm to (94.0, 60.8)
- moved R15 3.00 mm to (94.0, 64.0)
Connections:
- U9 pad 41_10: (no net) -> GNDREF
- U9 pad 41_11: (no net) -> GNDREF
- U9 pad 41_12: (no net) -> GNDREF
- U9 pad 41_13: (no net) -> GNDREF
- U9 pad 41_14: (no net) -> GNDREF
- U9 pad 41_15: (no net) -> GNDREF
- U9 pad 41_16: (no net) -> GNDREF
- U9 pad 41_17: (no net) -> GNDREF
- U9 pad 41_18: (no net) -> GNDREF
- U9 pad 41_19: (no net) -> GNDREF
- U9 pad 41_20: (no net) -> GNDREF
- U9 pad 41_21: (no net) -> GNDREF
Routing:
- net +3V3: track 123.9 -> 206.7 mm
- net /EN: track 10.0 -> 75.7 mm, vias 0 -> 2
- net GNDREF: track 20.3 -> 28.4 mm, vias 109 -> 163
- net +5V: track 20.6 -> 26.3 mm
- net Net-(D5-K): track 0.00 -> 3.99 mm
- net Net-(IC1-VDD18): track 0.00 -> 3.18 mm
- net /Pot1: track 11.3 -> 12.1 mm
- net /ENC_SW: track 50.4 -> 49.8 mm
- net /Pot2: track 34.1 -> 33.5 mm
- added copper zone on F.Cu, net GNDREF

Commit message: PCB finished
Parts:
- added J3: Conn_02x03_Counter_Clockwise, Connector_PinSocket_2.54mm:PinSocket_2x03_P2.54mm_Horizontal, F.Cu at (80.5, 97.9)
- added REF**: OSHW-Logo_7.5x8mm_SilkScreen, Symbol:OSHW-Logo_7.5x8mm_SilkScreen, F.Cu at (93.2, 62.5)
Connections:
- U9 pad 17: /NEOP -> unconnected-(U9-IO9-Pad17)
- U9 pad 34: unconnected-(U9-IO41-Pad34) -> /IO41
- U9 pad 35: unconnected-(U9-IO42-Pad35) -> /IO42
- U9 pad 38: unconnected-(U9-IO2-Pad38) -> /IO2
- U9 pad 39: unconnected-(U9-IO1-Pad39) -> /IO1
Routing:
- net GNDREF: track 28.4 -> 89.0 mm, vias 163 -> 362
- net /IO1: track 0.00 -> 12.4 mm
- net /IO2: track 0.00 -> 9.21 mm
- net +3V3: track 206.7 -> 214.6 mm
- net /IO41: track 0.00 -> 7.72 mm
- net /IO42: track 0.00 -> 5.34 mm
- net /IO0: track 63.3 -> 62.7 mm
- removed copper zone on F.Cu, net GNDREF
Other:
- board text added: "JLCJLCJLCJLC"
- board text added: "Supersonic Quantumbox v2.0 Adam Anderson 2023"
