File: Electronics/PCB/Supersonic Quantumbox/_autosave-Supersonic Quantumbox.kicad_sch (KiCad schematic)
At the start: 63 parts, among them IC1 AK4558EN, J1 USB_C_Receptacle_USB2.0, J2 Conn_01x12_Pin, J6 Barrel_Jack_Switch, SW1 RESET, SW2 BOOT, SW3 RotaryEncoder_Switch, SW4 SW_DPDT_x2, U1 Input_jack, U2 AZ1117-5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

Commit message: V2 schematic complete
Connections:
- no-connect marks 9 -> 12
Changed lines of the file:
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@@
   (junction (at 50.8 110.49) (diameter 0) (color 0 0 0 0)
   )
+  (no_connect (at 165.1 31.75))
+  (no_connect (at 283.21 152.4))
   (no_connect (at 196.85 25.4))
   (no_connect (at 217.17 25.4))
@@
   (no_connect (at 210.82 50.8))
   (no_connect (at 292.1 127))
+  (no_connect (at 280.67 30.48))
   (wire (pts (xy 284.48 142.24) (xy 292.1 142.24))
     (stroke (width 0) (type default))
@@
     )
   )
-  (symbol (lib_name "+3V3_1") (lib_id "power:+3V3") (at 201.93 119.38 0) (unit 1)
+  (symbol (lib_id "power:+3V3") (at 201.93 119.38 0) (unit 1)
     (in_bom yes) (on_board yes) (dnp no)
     (property "Reference" "#PWR012" (at 201.93 123.19 0)
@@
     )
   )
-  (symbol (lib_name "+3V3_1") (lib_id "power:+3V3") (at 153.67 162.56 0) (unit 1)
+  (symbol (lib_id "power:+3V3") (at 153.67 162.56 0) (unit 1)
     (in_bom yes) (on_board yes) (dnp no)
     (property "Reference" "#PWR030" (at 153.67 166.37 0)
@@
     )
   )
-  (symbol (lib_name "+3V3_1") (lib_id "power:+3V3") (at 167.64 106.68 0) (unit 1)
+  (symbol (lib_id "power:+3V3") (at 167.64 106.68 0) (unit 1)
     (in_bom yes) (on_board yes) (dnp no)
     (property "Reference" "#PWR031" (at 167.64 110.49 0)
@@
     )
   )
-  (symbol (lib_name "+3V3_1") (lib_id "power:+3V3") (at 152.4 109.22 0) (unit 1)
+  (symbol (lib_id "power:+3V3") (at 152.4 109.22 0) (unit 1)
     (in_bom yes) (on_board yes) (dnp no)
     (property "Reference" "#PWR011" (at 152.4 113.03 0)
